File: KiCad/3Way_valve_controller.kicad_sch (KiCad schematic)
At the start: 90 parts, among them J1 LCD 16x2, J2 USB_B_Mini, J6 Conn_01x12, Q1 2N7002, SW1 SW_Push, SW2 SW_Push, SW3 SW_Push, SW4 SW_Push, SW5 SW_Push, U1 PCF8574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

Commit message: Add files via upload
Parts:
- added C29: 10u, Capacitor_SMD:C_0805_2012Metric_Pad1.18x1.45mm_HandSolder, symbol Device:C
- added C30: 100n, Capacitor_SMD:C_0603_1608Metric, symbol Device:C
- added C31, C32: C, Capacitor_SMD:C_1206_3216Metric, symbol Device:C
- added C33, C34: C_Polarized, Capacitor_SMD:CP_Elec_10x10, symbol Device:C_Polarized
- added C35: 100n, Capacitor_SMD:C_0603_1608Metric_Pad1.08x0.95mm_HandSolder, symbol Device:C
- added L3: 4H7, Inductor_SMD:L_Bourns_SRP7028A_7.3x6.6mm, symbol Device:L
- added TP9: GND, TestPoint:TestPoint_Pad_D1.5mm, symbol Connector:TestPoint
- added U7: AP63205WU, Package_TO_SOT_SMD:TSOT-23-6, symbol Regulator_Switching:AP63205WU
- C20, C21: footprint Capacitor_SMD:C_0805_2012Metric_Pad1.18x1.45mm_HandSolder -> Capacitor_SMD:C_1206_3216Metric
- L2: value L -> 4H7
Connections:
- net +12V: now also C29.1, C33.1, U7.2 (EN), U7.3 (IN)
- net +5V: no longer J6.4 (Pin_4)
- net GND: now also C29.2, C31.2, C32.2, C33.2, C34.2, C35.1, TP9.1, U7.4 (GND)
- new net: C30.1, L3.1, U7.5 (SW)
- new net: C30.2, U7.6 (BST)
- new net +5P: C31.1, C32.1, C34.1, C35.2, J6.4 (Pin_4), L3.2, U7.1 (FB)
Other:
- moved on the sheet: C14, C15, C16, C17, C18, C19, C20, C21, C26, J1, L2, R13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

Commit message: Add files via upload
Parts:
- C18, C29: footprint Capacitor_SMD:C_0805_2012Metric_Pad1.18x1.45mm_HandSolder -> Capacitor_SMD:C_1206_3216Metric
Other:
- note removed: "end switches!!!"
Changed lines of the file:
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@@
 	(generator_version "9.0")
 	(paper "A3")
-	(text "end switches!!!\n"
-		(exclude_from_sim no)
-		(at 76.708 133.858 0)
-		(effects
-			(font
-				(size 1.27 1.27)
-			)
-		)
-	)
 	(text "Debug port"
 		(exclude_from_sim no)
@@
 			)
 		)
-		(property "Footprint" "Capacitor_SMD:C_0805_2012Metric_Pad1.18x1.45mm_HandSolder"
+		(property "Footprint" "Capacitor_SMD:C_1206_3216Metric"
 			(at 287.9852 81.28 0)
 			(effects
@@
 			)
 		)
-		(property "Footprint" "Capacitor_SMD:C_0805_2012Metric_Pad1.18x1.45mm_HandSolder"
+		(property "Footprint" "Capacitor_SMD:C_1206_3216Metric"
 			(at 305.7652 44.45 0)
 			(effects

Commit message: Add files via upload
Other:
- moved on the sheet: H2
Changed lines of the file:
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@@
 	(symbol
 		(lib_id "Mechanical:MountingHole")
-		(at 226.06 214.63 0)
+		(at 234.95 204.47 0)
 		(unit 1)
 		(exclude_from_sim no)
@@
 		(fields_autoplaced yes)
 		(property "Reference" "H2"
-			(at 228.6 213.3599 0)
+			(at 237.49 203.1999 0)
 			(effects
 				(font
@@
 		)
 		(property "Value" "MountingHole"
-			(at 228.6 215.8999 0)
+			(at 237.49 205.7399 0)
 			(effects
 				(font
@@
 		)
 		(property "Footprint" "MountingHole:MountingHole_3.2mm_M3"
-			(at 226.06 214.63 0)
+			(at 234.95 204.47 0)
 			(effects
 				(font
@@
 		)
 		(property "Datasheet" "~"
-			(at 226.06 214.63 0)
+			(at 234.95 204.47 0)
 			(effects
 				(font
@@
 		)
 		(property "Description" "Mounting Hole without connection"
-			(at 226.06 214.63 0)
+			(at 234.95 204.47 0)
 			(effects
 				(font
